File: new-anuduino-board.sch (KiCad schematic (older format))
At the start: 13 parts, among them IC1 ATTINY85-P, J1 USB_2, P1 CONN_4, P2 CONN_4

Commit message: a first backup, got scared, just had a dream
Connections:
- net D+: now reaches D1.2 (K), J1.2, R2.1
- net D-: now reaches D2.2 (K), J1.3, R1.2, R3.1
Changed lines of the file:
@@
-EESchema Schematic File Version 2  date Friday 28 March 2014 02:39:17 PM IST
+EESchema Schematic File Version 2  date Monday 31 March 2014 06:52:33 PM IST
 LIBS:power
 LIBS:device
@@
 Sheet 1 1
 Title ""
-Date "27 mar 2014"
+Date "31 mar 2014"
 Rev ""
 Comp ""
@@
 Comment4 ""
 $EndDescr
+Text Label 4850 3900 0    60   ~ 0
+D-
+Text Label 4850 3750 0    60   ~ 0
+D+
 Connection ~ 1800 3900
 Wire Wire Line
